File: pendo/pendo.kicad_pcb (KiCad board)
At the start: 4 copper layers, 140 x 67 mm, 52 parts, among them J1 Screw_Terminal_01x02, J3 Conn_01x04_Pin, J4 Conn_ARM_JTAG_SWD_10, J5 Conn_01x04_Pin, J6 Conn_01x04_Pin, J7 Conn_02x10_Odd_Even, J8 Conn_01x06_Pin, J9 Conn_01x06_Pin, SW1 SW_Push, SW2 SW_SPST, U1 STM32G431RBTx, U10 DRV8231ADSG, U11 DRV8231ADSG, U2 LSM6DS3, U4 ESP32-C3-WROOM-02, U5 AP2112K-3.3, U9 RPX-2.5-CT

Commit message: more routing
Parts:
- moved R5 18.0 mm to (117.7, 83.5)
- moved R7 12.7 mm to (117.0, 87.0)
- moved J8 12.5 mm to (107.5, 75.5), turned to 180 degrees
- moved C9 12.4 mm to (224.7, 81.0), turned to 0 degrees
- moved J9 9.75 mm to (218.2, 75.5)
- moved R6 7.14 mm to (183.5, 82.0), turned to 0 degrees
- moved C10 6.34 mm to (109.0, 79.5), turned to 180 degrees
- moved C11 4.99 mm to (220.0, 79.0)
- moved R1 4.72 mm to (103.0, 82.0)
- moved U10 4.00 mm to (106.5, 80.1), turned to 90 degrees
- moved U11 3.99 mm to (217.8, 80.0), turned to 90 degrees
- moved R2 3.95 mm to (214.5, 82.0)
- moved C18 3.81 mm to (109.0, 85.3)
- moved R4 2.15 mm to (182.5, 79.7), turned to 90 degrees
- moved C1 1.77 mm to (136.0, 98.8)
Connections:
- J3 pad 3: /I2C3_SDA -> /I2C1_SDA
- J3 pad 4: /I2C3_SCL -> /I2C1_SCL
- J5 pad 3: /I2C3_SDA -> /I2C1_SDA
- J5 pad 4: /I2C3_SCL -> /I2C1_SCL
- J6 pad 3: /I2C3_SDA -> /I2C1_SDA
- J6 pad 4: /I2C3_SCL -> /I2C1_SCL
- J7 pad 10: /I2C1_SCL -> /I2C3_SCL
- J7 pad 9: /I2C1_SDA -> /I2C3_SDA
Routing:
- net /ENC2A: track 0.00 -> 140.4 mm, vias 0 -> 2
- net /ENC2B: track 0.00 -> 89.4 mm
- net /I2C1_SDA: track 2.22 -> 58.5 mm, vias 0 -> 2
- net /I2C1_SCL: track 2.15 -> 56.2 mm, vias 0 -> 2
- net /TIM1_3: track 88.2 -> 141.8 mm
- net /TIM1_4: track 89.4 -> 141.5 mm
- net /ENC1B: track 0.00 -> 49.1 mm, vias 0 -> 2
- net /ENC1A: track 0.00 -> 47.3 mm, vias 0 -> 2
- net /PB12: track 0.00 -> 44.8 mm
- net /PB11: track 0.00 -> 44.4 mm
- net /E_STOP: track 0.00 -> 40.1 mm
- net +3.3V: track 10.4 -> 50.0 mm, vias 8 -> 15
- net /I2C3_SDA: track 7.51 -> 31.3 mm
- net /I2C3_SCL: track 7.30 -> 27.6 mm
- net Net-(U9-FB): track 2.14 -> 15.6 mm
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
Commit message: final production ready PCB complete with BOM and POS
Parts:
- removed C16, C17: 1u, Capacitor_SMD:C_0402_1005Metric
- removed U2: LSM6DS3, Package_LGA:LGA-14_3x2.5mm_P0.5mm_LayoutBorder3x4y
- added C23: 0.1u, Capacitor_SMD:C_0402_1005Metric, F.Cu at (140.0, 83.0)
- added C24: 1u, Capacitor_SMD:C_0402_1005Metric, F.Cu at (139.2, 81.6)
- added C25: 10n, Capacitor_SMD:C_0402_1005Metric, F.Cu at (139.5, 85.3)
- added D1: LED, LED_SMD:LED_0603_1608Metric, F.Cu at (194.2, 114.0)
- added D2: LED, LED_SMD:LED_0603_1608Metric, F.Cu at (175.0, 75.0)
- added D3: LED, LED_SMD:LED_0603_1608Metric, F.Cu at (194.2, 116.0)
- added G***: LOGO, Custom_Logos:rambutan, F.Cu at (222.0, 132.5)
- added J10: Conn_01x06_Pin, Connector_PinHeader_2.54mm:PinHeader_1x06_P2.54mm_Vertical, F.Cu at (106.0, 124.2)
- added R13: 1k, Resistor_SMD:R_1206_3216Metric, F.Cu at (197.0, 112.5)
- added R14: 300, Resistor_SMD:R_1206_3216Metric, F.Cu at (172.0, 76.5)
- added R15: 120, Resistor_SMD:R_1206_3216Metric, F.Cu at (197.0, 117.5)
- added U3: MPU-6500, footprints:QFN24_3X3X0P9_IVS, F.Cu at (136.8, 84.0)
- moved R7 16.7 mm to (109.0, 101.7), turned to 90 degrees
- moved R12 12.0 mm to (229.5, 106.0), turned to -90 degrees
- moved C5 7.24 mm to (229.5, 108.5), turned to -90 degrees
- moved J1 4.60 mm to (187.5, 107.0), turned to 0 degrees
- moved R5 3.95 mm to (119.5, 87.0), turned to 180 degrees
- moved U4 1.90 mm to (218.5, 103.5)
- moved C9 0.80 mm to (224.7, 81.8)
- renumbered J6 to I2C, J3 to I2C, J5 to I2C, J4 to JTAG, J8 to M1, J9 to M2, SW1 to RESET
Connections:
- U1 pad 36: unconnected-(U1-PB14-Pad36) -> /ENC_CS
Routing:
- net /VPROPI2: track 2.11 -> 139.6 mm, vias 0 -> 6
- net /ESP32_TX: track 0.00 -> 135.5 mm, vias 0 -> 4
- net /ESP32_RX: track 0.00 -> 132.1 mm, vias 0 -> 2
- net /JDB_SWDIO: track 11.0 -> 120.3 mm, vias 0 -> 2
- net /JDB_SWCLK: track 13.2 -> 122.2 mm, vias 0 -> 2
- net /JDB_RESET: track 94.3 -> 185.0 mm
- net /USART3_RX: track 0.00 -> 63.3 mm, vias 0 -> 1
- net /SPI1_MISO: track 6.55 -> 66.6 mm, vias 0 -> 5
- net /SPI1_MOSI: track 7.99 -> 66.1 mm, vias 0 -> 3
- net /USART3_TX: track 0.00 -> 55.9 mm, vias 0 -> 1
- net /SPI1_SCK: track 6.95 -> 60.4 mm, vias 1 -> 2
- net /SPI1_GP_CS1: track 0.00 -> 41.7 mm, vias 0 -> 1
- net /SPI1_GP_CS2: track 0.00 -> 39.3 mm, vias 0 -> 1
- net +3.3V: track 50.0 -> 85.8 mm, vias 15 -> 22
- net /ENC_CS: track 0.00 -> 31.6 mm, vias 0 -> 4
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Other:
- board text added: "12V"
- board text added: "3.3V"
- board text added: "5V"
- board text added: "CS"
- board text added: "GND"
- board text added: "KILL SWITCH"
- board text added: "MISO"
- board text added: "MOSI"
- board text added: "SCK"
- board text added: "SCL"
- board text added: "SDA"
- board text added: "SPI"
- board text added: "VIN"
