File: pendo/pendo.kicad_sch (KiCad schematic)
At the start: 52 parts, among them J1 Screw_Terminal_01x02, J3 Conn_01x04_Pin, J4 Conn_ARM_JTAG_SWD_10, J5 Conn_01x04_Pin, J6 Conn_01x04_Pin, J7 Conn_02x10_Odd_Even, J8 Conn_01x06_Pin, J9 Conn_01x06_Pin, SW1 SW_Push, SW2 SW_SPST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

Commit message: more routing
Connections:
- net I2C1_SCL: now also J3.4 (Pin_4), J5.4 (Pin_4), J6.4 (Pin_4); no longer J7.10 (Pin_10)
- net I2C1_SDA: now also J3.3 (Pin_3), J5.3 (Pin_3), J6.3 (Pin_3); no longer J7.9 (Pin_9)
- net I2C3_SCL: now also J7.10 (Pin_10); no longer J3.4 (Pin_4), J5.4 (Pin_4), J6.4 (Pin_4)
- net I2C3_SDA: now also J7.9 (Pin_9); no longer J3.3 (Pin_3), J5.3 (Pin_3), J6.3 (Pin_3)
Changed lines of the file:
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@@
 		)
 	)
-	(label "I2C1_SCL"
+	(label "I2C3_SCL"
 		(at 54.61 161.29 0)
 		(effects
@@
 		)
 	)
-	(label "I2C3_SDA"
+	(label "I2C1_SDA"
 		(at 240.03 151.13 0)
 		(effects
@@
 		)
 	)
-	(label "I2C3_SDA"
+	(label "I2C1_SDA"
 		(at 260.35 151.13 0)
 		(effects
@@
 		)
 	)
-	(label "I2C3_SCL"
+	(label "I2C1_SCL"
 		(at 260.35 148.59 0)
 		(effects
@@
 		)
 	)
-	(label "I2C3_SDA"
+	(label "I2C1_SDA"
 		(at 250.19 151.13 0)
 		(effects
@@
 		)
 	)
-	(label "I2C1_SDA"
+	(label "I2C3_SDA"
 		(at 36.83 161.29 180)
 		(effects
@@
 		)
 	)
-	(label "I2C3_SCL"
+	(label "I2C1_SCL"
 		(at 250.19 148.59 0)
 		(effects
@@
 		)
 	)
-	(label "I2C3_SCL"
+	(label "I2C1_SCL"
 		(at 240.03 148.59 0)
 		(effects

Commit message: final production ready PCB complete with BOM and POS
Parts:
- removed C16, C17: 1u, Capacitor_SMD:C_0402_1005Metric, symbol Device:C
- removed U2: LSM6DS3, Package_LGA:LGA-14_3x2.5mm_P0.5mm_LayoutBorder3x4y, symbol Sensor_Motion:LSM6DS3
- added C23: 0.1u, Capacitor_SMD:C_0402_1005Metric, symbol Device:C
- added C24: 1u, Capacitor_SMD:C_0402_1005Metric, symbol Device:C
- added C25: 10n, Capacitor_SMD:C_0402_1005Metric, symbol Device:C
- added D1, D2, D3: LED, LED_SMD:LED_0603_1608Metric, symbol Device:LED
- added J10: Conn_01x06_Pin, Connector_PinHeader_2.54mm:PinHeader_1x06_P2.54mm_Vertical, symbol Connector:Conn_01x06_Pin
- added R13: 1k, Resistor_SMD:R_1206_3216Metric, symbol Device:R_US
- added R14: 300, Resistor_SMD:R_1206_3216Metric, symbol Device:R_US
- added R15: 120, Resistor_SMD:R_1206_3216Metric, symbol Device:R_US
- added U3: MPU-6500, footprints:QFN24_3X3X0P9_IVS, symbol 2026-04-28_00-48-01:MPU-6500
Connections:
- net +12V: now also R13.1
- net +3.3V: now also C24.1, C25.1, J10.2 (Pin_2), R15.1, U3.13 (VDD), U3.8 (VDDIO)
- net +5V: now also R14.1
- net GND: now also C23.2, C24.2, C25.2, D1.2 (A), D2.2 (A), D3.2 (A), J10.1 (Pin_1), U3.18 (GND)
- net IMU_CS: now also U3.22 (nCS)
- net IMU_INT: now also U3.12 (INT)
- net SPI1_MISO: now also J10.4 (Pin_4), U3.9 (SDO/ADO)
- net SPI1_MOSI: now also J10.3 (Pin_3), U3.24 (SDA/SDI)
- net SPI1_SCK: now also J10.5 (Pin_5), U3.23 (SCL/SCLK)
- net ENC_CS: now reaches U1.36 (PB14)
- net ENC_CS: now also J10.6 (Pin_6)
- new net: D3.1 (K), R15.2
- new net: D2.1 (K), R14.2
- new net: D1.1 (K), R13.2
- new net: C23.1, U3.10 (REGOUT)
- no-connect marks 36 -> 34
Other:
- note added: "Encoder SPI"
- moved on the sheet: J7
